File: macro20.sch (KiCad schematic (older format))
At the start: 5 parts, among them J1 Conn_01x04_Female, J2 Conn_01x03_Male, SW1 SW_Push, U1 ProMicro

Commit message: Update board
Connections:
- net VCC: now also J2.1 (Pin_1)
- net at U1.24 (RAW): no longer J2.1 (Pin_1)
Changed lines of the file:
@@
 	6800 3900 6300 3900
-Wire Wire Line
-	5650 2800 7050 2800
 Wire Wire Line
 	5850 2900 5850 2600
@@
 Wire Wire Line
 	6000 3900 5650 3900
+Text GLabel 7050 2800 0    50   UnSpc ~ 0
+VCC
 $EndSCHEMATC
