File: macro20.kicad_pcb (KiCad board)
At the start: 2 copper layers, 98.4 x 98.4 mm, 51 parts, among them J1 Conn_01x04_Female, J2 Conn_01x03_Male, SW1 SW_Push, U1 ProMicro

Commit message: Update board
Connections:
- J2 pad 1: Net-(J2-Pad1) -> VCC
- U1 pad 24: Net-(J2-Pad1) -> Net-(U1-Pad24)
Routing:
- net Net-(J2-Pad1): track 52.6 -> 0.00 mm
- net VCC: track 30.5 -> 49.2 mm
Changed lines of the file:
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@@
-(kicad_pcb (version 20171130) (host pcbnew 5.1.5)
+(kicad_pcb (version 20171130) (host pcbnew "(5.1.5)-3")
   (general
     (thickness 1.6)
     (drawings 19)
-    (tracks 230)
+    (tracks 231)
     (zones 0)
     (modules 51)
@@
   (net 38 "Net-(J1-Pad2)")
   (net 39 GND)
-  (net 40 "Net-(J2-Pad1)")
-  (net 41 "Net-(J2-Pad2)")
-  (net 42 "Net-(SW1-Pad2)")
-  (net 43 "Net-(R1-Pad2)")
+  (net 40 "Net-(J2-Pad2)")
+  (net 41 "Net-(SW1-Pad2)")
+  (net 42 "Net-(R1-Pad2)")
+  (net 43 "Net-(U1-Pad24)")
   (net_class Default "This is the default net class."
     (clearance 0.2)
@@
     (add_net "Net-(J1-Pad1)")
     (add_net "Net-(J1-Pad2)")
-    (add_net "Net-(J2-Pad1)")
     (add_net "Net-(J2-Pad2)")
     (add_net "Net-(R1-Pad2)")
@@
     (add_net "Net-(U1-Pad16)")
     (add_net "Net-(U1-Pad2)")
+    (add_net "Net-(U1-Pad24)")
     (add_net "Net-(U1-Pad7)")
     (add_net ROW1)
@@
     (fp_line (start 15.24 -8.89) (end 15.24 8.89) (layer B.SilkS) (width 0.15))
     (pad 24 thru_hole circle (at -13.97 -7.62 270) (size 1.6 1.6) (drill 1.1) (layers *.Cu *.Mask F.SilkS)
-      (net 40 "Net-(J2-Pad1)"))
+      (net 43 "Net-(U1-Pad24)"))
     (pad 23 thru_hole circle (at -11.43 -7.62 270) (size 1.6 1.6) (drill 1.1) (layers *.Cu *.Mask F.SilkS)
       (net 39 GND))
     (pad 22 thru_hole circle (at -8.89 -7.62 270) (size 1.6 1.6) (drill 1.1) (layers *.Cu *.Mask F.SilkS)
-      (net 42 "Net-(SW1-Pad2)"))
+      (net 41 "Net-(SW1-Pad2)"))
     (pad 21 thru_hole circle (at -6.35 -7.62 270) (size 1.6 1.6) (drill 1.1) (layers *.Cu *.Mask F.SilkS)
       (net 36 VCC))
@@
       (net 32 "Net-(U1-Pad14)"))
     (pad 13 thru_hole circle (at 13.97 -7.62 270) (size 1.6 1.6) (drill 1.1) (layers *.Cu *.Mask F.SilkS)
-      (net 43 "Net-(R1-Pad2)"))
+      (net 42 "Net-(R1-Pad2)"))
     (pad 12 thru_hole circle (at 13.97 7.62 270) (size 1.6 1.6) (drill 1.1) (layers *.Cu *.Mask F.SilkS)
       (net 10 ROW5))
@@
     (fp_line (start 0.74 0.8) (end 0.74 -0.8) (layer B.Fab) (width 0.1))
     (pad 2 thru_hole oval (at 5.08 0) (size 1.4 1.4) (drill 0.7) (layers *.Cu *.Mask)
-      (net 43 "Net-(R1-Pad2)"))
+      (net 42 "Net-(R1-Pad2)"))
     (pad 1 thru_hole circle (at 0 0) (size 1.4 1.4) (drill 0.7) (layers *.Cu *.Mask)
-      (net 41 "Net-(J2-Pad2)"))
+      (net 40 "Net-(J2-Pad2)"))
     (model ${KISYS3DMOD}/Resistor_THT.3dshapes/R_Axial_DIN0204_L3.6mm_D1.6mm_P5.08mm_Horizontal.wrl
       (at (xyz 0 0 0))
@@
       (net 39 GND))
     (pad 2 thru_hole circle (at 6.5 4.5 90) (size 2 2) (drill 1.1) (layers *.Cu *.Mask)
-      (net 42 "Net-(SW1-Pad2)"))
+      (net 41 "Net-(SW1-Pad2)"))
     (pad 1 thru_hole circle (at 0 0 90) (size 2 2) (drill 1.1) (layers *.Cu *.Mask)
       (net 39 GND))
     (pad 2 thru_hole circle (at 0 4.5 90) (size 2 2) (drill 1.1) (layers *.Cu *.Mask)
-      (net 42 "Net-(SW1-Pad2)"))
+      (net 41 "Net-(SW1-Pad2)"))
     (model ${KISYS3DMOD}/Button_Switch_THT.3dshapes/SW_PUSH_6mm.wrl
       (at (xyz 0 0 0))
@@
       (net 39 GND))
     (pad 2 thru_hole oval (at 0 -2.54) (size 1.7 1.7) (drill 1) (layers *.Cu *.Mask)
-      (net 41 "Net-(J2-Pad2)"))
+      (net 40 "Net-(J2-Pad2)"))
     (pad 1 thru_hole rect (at 0 0) (size 1.7 1.7) (drill 1) (layers *.Cu *.Mask)
-      (net 40 "Net-(J2-Pad1)"))
+      (net 36 VCC))
     (model ${KISYS3DMOD}/Connector_PinHeader_2.54mm.3dshapes/PinHeader_1x03_P2.54mm_Vertical.wrl
       (at (xyz 0 0 0))
@@
   (segment (start 160.014213 114.3) (end 165.1 114.3) (width 0.25) (layer B.Cu) (net 39))
   (segment (start 158.6 114.3) (end 160.014213 114.3) (width 0.25) (layer B.Cu) (net 39))
-  (segment (start 167.005 57.15) (end 163.83 53.975) (width 0.25) (layer F.Cu) (net 40))
-  (segment (start 167.005 97.62) (end 167.005 57.15) (width 0.25) (layer F.Cu) (net 40))
-  (segment (start 161.29 102.235) (end 162.39 102.235) (width 0.25) (layer F.Cu) (net 40))
-  (segment (start 162.39 102.235) (end 167.005 97.62) (width 0.25) (layer F.Cu) (net 40))
-  (segment (start 161.29 99.695) (end 160.087919 99.695) (width 0.25) (layer F.Cu) (net 41))
-  (segment (start 160.087919 99.695) (end 159.385 98.992081) (width 0.25) (layer F.Cu) (net 41))
-  (segment (start 159.385 92.355051) (end 159.385 94.615) (width 0.25) (layer F.Cu) (net 41))
-  (segment (start 158.115 92.075) (end 159.104949 92.075) (width 0.25) (layer F.Cu) (net 41))
-  (segment (start 159.385 98.992081) (end 159.385 94.615) (width 0.25) (layer F.Cu) (net 41))
-  (segment (start 159.104949 92.075) (end 159.385 92.355051) (width 0.25) (layer F.Cu) (net 41))
-  (segment (start 159.385 94.615) (end 159.385 93.98) (width 0.25) (layer F.Cu) (net 41))
-  (via (at 165.1 97.79) (size 0.8) (drill 0.4) (layers F.Cu B.Cu) (net 42))
-  (segment (start 163.83 59.055) (end 165.1 60.325) (width 0.25) (layer F.Cu) (net 42))
-  (segment (start 165.1 60.325) (end 165.1 97.79) (width 0.25) (layer F.Cu) (net 42))
-  (segment (start 161.29 113.03) (end 161.29 116.11) (width 0.25) (layer F.Cu) (net 42))
-  (segment (start 162.505 116.205) (end 161.29 116.205) (width 0.25) (layer F.Cu) (net 42))
-  (segment (start 165.1 118.8) (end 162.505 116.205) (width 0.25) (layer F.Cu) (net 42))
-  (segment (start 161.29 116.11) (end 161.29 116.205) (width 0.25) (layer F.Cu) (net 42))
-  (segment (start 161.29 116.205) (end 158.6 118.8) (width 0.25) (layer F.Cu) (net 42))
-  (via (at 165.1 101.6) (size 0.8) (drill 0.4) (layers F.Cu B.Cu) (net 42))
-  (segment (start 165.1 97.79) (end 165.1 101.6) (width 0.25) (layer B.Cu) (net 42))
-  (segment (start 165.1 109.22) (end 161.29 113.03) (width 0.25) (layer F.Cu) (net 42))
-  (segment (start 165.1 101.6) (end 165.1 109.22) (width 0.25) (layer F.Cu) (net 42))
-  (segment (start 163.195 82.55) (end 163.83 81.915) (width 0.25) (layer F.Cu) (net 43))
-  (segment (start 163.195 92.075) (end 163.195 82.55) (width 0.25) (layer F.Cu) (net 43))
+  (segment (start 161.29 102.235) (end 162.39 102.235) (width 0.25) (layer F.Cu) (net 36))
+  (segment (start 156.630001 88.479999) (end 157.48 87.63) (width 0.25) (layer F.Cu) (net 36))
+  (segment (start 156.630001 98.675001) (end 156.630001 88.479999) (width 0.25) (layer F.Cu) (net 36))
+  (segment (start 160.19 102.235) (end 156.630001 98.675001) (width 0.25) (layer F.Cu) (net 36))
+  (segment (start 161.29 102.235) (end 160.19 102.235) (width 0.25) (layer F.Cu) (net 36))
+  (segment (start 161.29 99.695) (end 160.087919 99.695) (width 0.25) (layer F.Cu) (net 40))
+  (segment (start 160.087919 99.695) (end 159.385 98.992081) (width 0.25) (layer F.Cu) (net 40))
+  (segment (start 159.385 92.355051) (end 159.385 94.615) (width 0.25) (layer F.Cu) (net 40))
+  (segment (start 158.115 92.075) (end 159.104949 92.075) (width 0.25) (layer F.Cu) (net 40))
+  (segment (start 159.385 98.992081) (end 159.385 94.615) (width 0.25) (layer F.Cu) (net 40))
+  (segment (start 159.104949 92.075) (end 159.385 92.355051) (width 0.25) (layer F.Cu) (net 40))
+  (segment (start 159.385 94.615) (end 159.385 93.98) (width 0.25) (layer F.Cu) (net 40))
+  (via (at 165.1 97.79) (size 0.8) (drill 0.4) (layers F.Cu B.Cu) (net 41))
+  (segment (start 163.83 59.055) (end 165.1 60.325) (width 0.25) (layer F.Cu) (net 41))
+  (segment (start 161.29 113.03) (end 161.29 116.11) (width 0.25) (layer F.Cu) (net 41))
+  (segment (start 162.505 116.205) (end 161.29 116.205) (width 0.25) (layer F.Cu) (net 41))
+  (segment (start 165.1 118.8) (end 162.505 116.205) (width 0.25) (layer F.Cu) (net 41))
+  (segment (start 161.29 116.11) (end 161.29 116.205) (width 0.25) (layer F.Cu) (net 41))
+  (segment (start 161.29 116.205) (end 158.6 118.8) (width 0.25) (layer F.Cu) (net 41))
+  (via (at 165.1 101.6) (size 0.8) (drill 0.4) (layers F.Cu B.Cu) (net 41))
+  (segment (start 165.1 97.79) (end 165.1 101.6) (width 0.25) (layer B.Cu) (net 41))
+  (segment (start 165.1 109.22) (end 161.29 113.03) (width 0.25) (layer F.Cu) (net 41))
+  (segment (start 165.1 101.6) (end 165.1 109.22) (width 0.25) (layer F.Cu) (net 41))
+  (segment (start 165.1 60.325) (end 165.1 97.79) (width 0.25) (layer F.Cu) (net 41))
+  (segment (start 163.195 82.55) (end 163.83 81.915) (width 0.25) (layer F.Cu) (net 42))
+  (segment (start 163.195 92.075) (end 163.195 82.55) (width 0.25) (layer F.Cu) (net 42))
   (zone (net 39) (net_name GND) (layer B.Cu) (hatch edge 0.508)
     (connect_pads (clearance 0.508))

Commit message: Silkscreen/mask graphics
Parts:
- added REF**: OSHW-Symbol_8.9x8mm_Mask, logo:OSHW-Symbol_8.9x8mm_Mask, B.Cu at (163.2, 128.9)
Other:
- board text added: "github.com/JB6a62"

Commit message: Silkscreen/mask changes
Other:
- board text added: "macro20"
- board text added: "rev 1.0"
- board text removed: "RAW"
- board text removed: "REV 1.0"
Changed lines of the file:
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@@
   (general
     (thickness 1.6)
-    (drawings 20)
+    (drawings 21)
     (tracks 231)
     (zones 0)
@@
     )
   )
-  (gr_text github.com/JB6a62 (at 146.685 128.905) (layer B.Mask)
+  (gr_text macro20 (at 158.75 146.05) (layer B.SilkS)
+    (effects (font (size 1 1) (thickness 0.15)) (justify mirror))
+  )
+  (gr_text github.com/JB6a62 (at 146.685 128.905) (layer B.SilkS)
     (effects (font (size 1.5 1.5) (thickness 0.2)) (justify mirror))
   )
-  (gr_text "REV 1.0" (at 160.02 146.05) (layer B.SilkS)
+  (gr_text "rev 1.0" (at 149.86 146.05) (layer B.SilkS)
     (effects (font (size 1 1) (thickness 0.15)) (justify mirror))
   )
-  (gr_text JLCJLCJLCJLC (at 147.955 146.05) (layer B.SilkS)
+  (gr_text JLCJLCJLCJLC (at 138.43 146.05) (layer B.SilkS)
     (effects (font (size 1 1) (thickness 0.15)) (justify mirror))
   )
@@
     (effects (font (size 1 1) (thickness 0.15)) (justify mirror))
   )
-  (gr_text RAW (at 158.115 102.235) (layer B.SilkS)
+  (gr_text VCC (at 158.115 102.235) (layer B.SilkS)
     (effects (font (size 1 1) (thickness 0.15)) (justify mirror))
   )
